Commit message: Attached all 4 ailerons to rocket, FIXME's regarding that in code; finalized environment/colors; set-up controls for 4 ailerons, physics changes required

File: LRI_Meshcat/Implementation/urdf/ground.urdf (robot description, URDF)
Before this commit: robot ground, 1 links, 0 joints
Links:
- link ground: geometry collision mesh filename=ground.stl scale=100 100 1; visual mesh filename=ground.stl scale=100 100 1

File: LRI_Meshcat/Implementation/urdf/rocket.urdf (robot description, URDF)
Before this commit: robot flying-wing, 3 links, 2 joints
Links:
- removed link aileron_left
- removed link aileron_right
- added link aileron1, mass 0.05; collision mesh filename=aileron1.stl; visual mesh filename=aileron1.stl
- added link aileron2, mass 0.05; collision mesh filename=aileron2.stl; visual mesh filename=aileron2.stl
- added link aileron3, mass 0.05; collision mesh filename=aileron3.stl; visual mesh filename=aileron3.stl
- added link aileron4, mass 0.05; collision mesh filename=aileron4.stl; visual mesh filename=aileron4.stl
Joints:
- removed joint left_aileron_joint
- removed joint right_aileron_joint
- added joint aileron1_joint: type revolute, parent base, child aileron1, origin xyz=0.5 0.3 0.0 rpy=0 0 0, axis 0 1 0, limit lower=-0.5 upper=0.5 effort=1 velocity=1
- added joint aileron2_joint: type revolute, parent base, child aileron2, origin xyz=0.5 -0.3 0.0 rpy=0 0 3.1416, axis 0 1 0, limit lower=-0.5 upper=0.5 effort=1 velocity=1
- added joint aileron3_joint: type revolute, parent base, child aileron3, origin xyz=-0.5 0.0 0.0 rpy=0 0 1.5708, axis 0 1 0, limit lower=-0.5 upper=0.5 effort=1 velocity=1
- added joint aileron4_joint: type revolute, parent base, child aileron4, origin xyz=0.0 0.5 0.0 rpy=0 0 -1.5708, axis 0 1 0, limit lower=-0.5 upper=0.5 effort=1 velocity=1
